File: sesame.sch (KiCad schematic (older format))
At the start: 155 parts, among them U1 ATmega32A-PU

Commit message: Use components more in line with other similar kits (Mysterium etc.)
Parts:
- R2, R3: value 68R -> 75R
- USB1: symbol Connector:USB_C_Receptacle_USB2.0 -> sesame-rescue:USB_C_Receptacle_USB2.0-Connector
Changed lines of the file:
@@
 P 8350 5600
 F 0 "R3" V 8250 5600 50  0000 C CNN
-F 1 "68R" V 8350 5600 50  0000 C CNN
+F 1 "75R" V 8350 5600 50  0000 C CNN
 F 2 "Resistor_THT:R_Axial_DIN0207_L6.3mm_D2.5mm_P10.16mm_Horizontal" V 8280 5600 50  0001 C CNN
 F 3 "~" H 8350 5600 50  0001 C CNN
@@
 P 8350 5400
 F 0 "R2" V 8450 5400 50  0000 C CNN
-F 1 "68R" V 8350 5400 50  0000 C CNN
+F 1 "75R" V 8350 5400 50  0000 C CNN
 F 2 "Resistor_THT:R_Axial_DIN0207_L6.3mm_D2.5mm_P10.16mm_Horizontal" V 8280 5400 50  0001 C CNN
 F 3 "~" H 8350 5400 50  0001 C CNN
@@
 	10150 5200 10250 5200
 $Comp
-L Connector:USB_C_Receptacle_USB2.0 USB1
+L sesame-rescue:USB_C_Receptacle_USB2.0-Connector USB1
 U 1 1 5F2A909F
 P 6450 5500
